File: Tinycam_v1/Tinycam_v1.kicad_sch (KiCad schematic)
At the start: 53 parts, among them J1 USB_C_Receptacle_USB2.0, J2 Micro_SD_Card, J7 LW05201-18 FPC Connector, Q1 SI2302, Q2 AO3400A, Q3 SS8050, Q4 SS8050, U1 IP4234CZ6, U2 ESP32-S3-WROOM-1, U3 ST1S12XX, U4 XC6219B152MR, U5 XC6219B282MR, Y1 DSX321G 24 MHZ

Commit message: .
Parts:
- removed C4: 10uF, Capacitor_SMD:C_0603_1608Metric, symbol Device:C_Small
- removed C5, C6, C7: 100n, Capacitor_SMD:C_0402_1005Metric_Pad0.74x0.62mm_HandSolder, symbol Device:C_Small
- removed CAM1: OV5640, _conn:CAM_OV5640_OMRON_XF2M-2415-1A, symbol _sensors:CAM_OV5640
- removed J7: LW05201-18 FPC Connector, _conn:Conn_FPC_LW05201-18, symbol Connector:Conn_01x18_Socket
- removed OSC_TYPE1: OSC_IN/EX, Jumper:SolderJumper-3_P1.3mm_Open_RoundedPad1.0x1.5mm_NumberLabels, symbol Jumper:Jumper_3_Open
- removed Q1: SI2302, Package_TO_SOT_SMD:SOT-23, symbol Device:Q_NMOS_GSD
- removed Q2: AO3400A, Package_TO_SOT_SMD:SOT-23, symbol Transistor_FET:AO3400A
- removed Q3, Q4: SS8050, Package_TO_SOT_SMD:SOT-23, symbol Device:Q_NPN_BCE
- removed R15: 150, Resistor_SMD:R_0402_1005Metric, symbol Device:R
- removed R16: 10K, Resistor_SMD:R_0402_1005Metric, symbol Device:R
- removed R17: 27.4, Resistor_SMD:R_0402_1005Metric, symbol Device:R
- removed R4, R5: 4.7k, Resistor_SMD:R_0402_1005Metric_Pad0.72x0.64mm_HandSolder, symbol Device:R
- removed R6, R9: 10k, Resistor_SMD:R_0402_1005Metric_Pad0.72x0.64mm_HandSolder, symbol Device:R
- removed R7, R8: 5.1k, Resistor_SMD:R_0402_1005Metric_Pad0.72x0.64mm_HandSolder, symbol Device:R
- removed U2: ESP32-S3-WROOM-1, RF_Module:ESP32-S3-WROOM-1, symbol RF_Module:ESP32-S3-WROOM-1
- removed Y1: DSX321G 24 MHZ, Crystal:Crystal_SMD_3225-4Pin_3.2x2.5mm_HandSoldering, symbol Device:Crystal_GND24
- added C15, C17: 10uF, Capacitor_SMD:C_0603_1608Metric_Pad1.08x0.95mm_HandSolder, symbol Device:C_Small
- added C16, C18, C19, C20: 100n, Capacitor_SMD:C_0402_1005Metric_Pad0.74x0.62mm_HandSolder, symbol Device:C_Small
- added J3: FFC/FPC 1mm 15pin MIPI-CSI, symbol Connector:Conn_01x15_Socket
- added J4: FFC/FPC 1mm 15pin MIPI-DSI, symbol Connector:Conn_01x15_Socket
- added J5: ESP32-C6 JTAG, symbol Connector_Generic:Conn_02x05_Odd_Even
- added J6: Display OSPTEK AM200Q460460LK, _conn:Conn_OK-14F024-04, symbol Connector:Conn_01x24_Socket
- added JP1: VBATor3v3, Jumper:SolderJumper-3_P1.3mm_Open_RoundedPad1.0x1.5mm_NumberLabels, symbol Jumper:Jumper_3_Open
- added Q5, Q6: SS8050, Package_TO_SOT_SMD:SOT-23, symbol Transistor_BJT:SS8050
- added R20, R21, R22: 10k, Resistor_SMD:R_0402_1005Metric_Pad0.72x0.64mm_HandSolder, symbol Device:R_Small
- added R23: 10K, Resistor_SMD:R_0402_1005Metric, symbol Device:R
- added SW1, SW2: SW_Push, _buttons:SW_SMD_KLS7-TS3401, symbol Switch:SW_Push
- added U6: ESP32-P4_MODULE, _chips:ESP32-P4_MODULE, symbol _MK:ESP32-P4_MODULE
Connections:
- net +3.3V: now also C15.1, C16.1, C17.1, C18.1, J3.15 (Pin_15), J4.14 (Pin_14), J4.15 (Pin_15), J5.1 (Pin_1), R20.2, R21.2, R22.2, R23.1
- net EN: now also Q5.3 (C)
- net FLASH: now also Q6.2 (E)
- net GND: now also C15.2, C16.2, C17.2, C18.2, C19.2, C20.2, J3.1 (Pin_1), J3.10 (Pin_10), J3.4 (Pin_4), J3.7 (Pin_7), J4.1 (Pin_1), J4.10 (Pin_10), J4.13 (Pin_13), J4.4 (Pin_4), J4.7 (Pin_7), J5.3 (Pin_3), J5.5 (Pin_5), J5.7 (Pin_7), J5.9 (Pin_9), J6.10 (Pin_10), J6.16 (Pin_16), J6.21 (Pin_21), SW1.2, SW2.1, U6.1 (GND), U6.15 (GND), U6.3 (GND), U6.33 (GND), U6.40 (GND), U6.47 (GND), U6.52 (GND), U6.83 (GND)
- net GPIO0: now also Q6.3 (C)
- net RESET: now also Q5.2 (E)
- net SD_DET: now reaches J2.S (Switch), R13.2, R14.2
- net at R18.1: now also Q5.1 (B)
- net at R19.1: now also Q6.1 (B)
- net SD_D2: now reaches J2.1 (DAT2)
- net SD_D2: now also U6.69 (GPIO41)
- net SD_D1: now reaches J2.8 (DAT1)
- net SD_D1: now also U6.68 (GPIO40)
- net MISO renamed SD_D0
- net SD_D0: now also U6.67 (GPIO39)
- net MOSI renamed SD_CMD
- net SD_CMD: now also U6.72 (GPIO44)
- net SCK renamed SD_CLK
- net SD_CLK: now also U6.71 (GPIO43)
- net SD_CS renamed SD_D3
- net SD_D3: now also U6.70 (GPIO42)
- new net: C20.1, R22.1, SW2.2, U6.87 (ESP_EN)
- new net: C19.1, R20.1, SW1.1, U6.62 (GPIO35/BOOT)
- new net: J6.15 (Pin_15), JP1.2 (C)
- new net: R21.1, U6.63 (GPIO36/BOOT_EN)
- new net +BATT: JP1.1 (A)
- new net AMOLED_CS: J6.7 (Pin_7)
- new net AMOLED_CTP_INT: J6.17 (Pin_17)
- new net AMOLED_CTP_RST: J6.18 (Pin_18)
- new net AMOLED_CTP_SCL: J6.19 (Pin_19)
- new net AMOLED_CTP_SDA: J6.20 (Pin_20)
- new net AMOLED_QSPI_CLK: J6.6 (Pin_6)
- new net AMOLED_QSPI_SI00: J6.5 (Pin_5)
- new net AMOLED_QSPI_SI01: J6.4 (Pin_4)
- new net AMOLED_QSPI_SI02: J6.3 (Pin_3)
- new net AMOLED_QSPI_SI03: J6.2 (Pin_2)
- new net AMOLED_RST: J6.8 (Pin_8)
- new net AMOLED_TE: J6.9 (Pin_9)
- new net AMOLED_VCI_EN: J6.1 (Pin_1), J6.13 (Pin_13), J6.14 (Pin_14), J6.22 (Pin_22), J6.23 (Pin_23), JP1.3 (B), R23.2
- new net C6_TCK: J5.4 (Pin_4), U6.12 (C6_IO6/MTCK)
- new net C6_TDI: J5.8 (Pin_8), U6.13 (C6_IO5/MTDI)
- new net C6_TDO: J5.6 (Pin_6), U6.11 (C6_IO7/MTDO)
- new net C6_TMS: J5.2 (Pin_2), U6.14 (C6_IO4/MTMS)
- new net CAM_CLK_N: J3.8 (Pin_8), U6.44 (CSI_CLKN)
- new net CAM_CLK_P: J3.9 (Pin_9), U6.43 (CSI_CLKP)
- new net CAM_D0_N: J3.2 (Pin_2), U6.41 (CSI_DATAN0)
- new net CAM_D0_P: J3.3 (Pin_3), U6.42 (CSI_DATAP0)
- new net CAM_D1_N: J3.5 (Pin_5), U6.45 (CSI_DATAN1)
- new net CAM_D1_P: J3.6 (Pin_6), U6.46 (CSI_DATAP1)
- new net CAM_IO0_PwEN: J3.11 (Pin_11)
- new net CAM_IO1_LED: J3.12 (Pin_12)
- new net DISP_CLK_N: J4.5 (Pin_5), U6.36 (DSI_CLKN)
- new net DISP_CLK_P: J4.6 (Pin_6), U6.37 (DSI_CLKP)
- new net DISP_D0_N: J4.8 (Pin_8), U6.39 (DSI_DATAN0)
- new net DISP_D0_P: J4.9 (Pin_9), U6.38 (DSI_DATAP0)
- new net DISP_D1_N: J4.2 (Pin_2), U6.35 (DSI_DATAN1)
- new net DISP_D1_P: J4.3 (Pin_3), U6.34 (DSI_DATAP1)
- new net ESP_3V3: U6.85 (ESP_3V3), U6.86 (ESP_3V3)
- new net I2C_SCL: J3.13 (Pin_13), J4.11 (Pin_11)
- new net I2C_SDA: J3.14 (Pin_14), J4.12 (Pin_12)
- new net USBFS1_D+: U6.51 (GPIO25/USB1P1_P0)
- new net USBFS1_D-: U6.50 (GPIO24/USB1P1_N0)
- new net USBFS2_D+: U6.54 (GPIO27/USB1P1_P1)
- new net USBFS2_D-: U6.53 (GPIO26/USB1P1_N1)
- new net USBHS_D+: U6.49 (USB_DP)
- new net USBHS_D-: U6.48 (USB_DM)
- no-connect marks 10 -> 9
Other:
- note added: "CSI - 100 Ohm DSI - 100 Ohm USB - 90 Ohm ANT - 50 Ohm"
- note added: "FS"
- note added: "HS"
- note added: "Waveshare ESP32-P4 module"
- note removed: "Avoid touching while resetting the MCU"
- note removed: "DFRobot AI CAM"
- note removed: "ESP32-S3-N16R8"
- note removed: "OV5640 camera breakouts https://wiki.dfrobot.com/SKU_DFR1154_ESP32_S3_AI_CAM#3.1%20Arduino%20IDE%20Configuration https://learn.adafruit.com/adafruit-ov5640-camera-breakout/downloads"
- note removed: "PSRAM IS USED"
- note removed: "https://github.com/koendv/cst816t/blob/master/extras/Schematic_drawing_2023-06-21.pdf https://www.lcsc.com/product-detail/FFC-FPC-Connectors_MINTRON-LW05201-18_C375900.html https://aliexpress.ru/item/1005005666658833.html?sku_id=12000037965813214"
- moved on the sheet: C10, C11, C12, C13, C14, C8, C9, D3, J2, L1, R10, R11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
