File: KICAD_Tinycam_v1/_restore_backup_2026-07-18T15-57-00-753/snapshots/KICAD_Tinycam_v1_snapshot_stepmanual_before_gpio_wiring_20260710_182228/Tinycam_v1.kicad_sch (KiCad schematic)
At the start: 51 parts, among them J1 USB_C_Receptacle_USB2.0, J2 Micro_SD_Card, J3 FFC/FPC 1mm 15pin MIPI-CSI, J4 FFC/FPC 1mm 15pin MIPI-DSI, J5 ESP32-C6 JTAG, J6 Display OSPTEK AM200Q460460LK, Q5 SS8050, Q6 SS8050, SW1 SW_Push, SW2 SW_Push, U1 IP4234CZ6, U3 ST1S12XX, U4 XC6219B152MR, U5 XC6219B282MR, U6 ESP32-P4_MODULE

Commit message: .
Parts:
- added J7: Conn_01x31_Socket, symbol Connector:Conn_01x31_Socket
- added JP2: VBATor3v3, Jumper:SolderJumper-3_P1.3mm_Open_RoundedPad1.0x1.5mm_NumberLabels, symbol Jumper:Jumper_3_Open
Other:
- moved on the sheet: C10, C11, C12, C13, C14, C15, C16, C17, C18, C8, C9, J3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
